Commit message: Add files via upload

File: src/my_robot_description/urdf/mobile_base.xacro (robot description, xacro)
@@ -129,7 +129,7 @@
         </collision>
         <inertial>
-            <mass value="1e-5" />
-            <origin xyz="0 0 0" rpy="0 0 0"/>
-            <inertia ixx="1e-6" ixy="0" ixz="0" iyy="1e-6" iyz="0" izz="1e-6" />
+          <mass value="1e-5" />
+          <origin xyz="0 0 0" rpy="0 0 0" />
+          <inertia ixx="4.05e-11" ixy="0" ixz="0" iyy="4.05e-11" iyz="0" izz="4.05e-11" />
         </inertial>
     </link>

File: src/my_robot_description/urdf/mobile_base_gazebo.xacro (robot description, xacro)
@@ -39,42 +39,43 @@
     </plugin>
   </gazebo>
+   <!--Laser -->
   <gazebo reference="Laser_link">
-    <material>Gazebo/Red</material>
-    <sensor name="laser" type="ray">
-        <pose> 0 0 0 0 0 0 </pose>
-        <visualize>true</visualize>
-        <update_rate>10</update_rate>
-        <ray>
-            <scan>
-                <horizontal>
-                    <samples>360</samples>
-                    <min_angle>-3.14</min_angle>
-                    <max_angle>3.14</max_angle>
-                </horizontal>
-            </scan>
-            <range>
-                <min>0.3</min>
-                <max>12</max>
-            </range>
-        </ray>
-        <plugin name="laser_controller" filename="libgazebo_ros_ray_sensor.so">
-            <ros>
-                <argument>~/out:=scan</argument>
-            </ros>
-            <output_type>sensor_msgs/LaserScan</output_type>
-            <frame_name>Laser_link</frame_name>
-        </plugin>
-    </sensor>
-</gazebo>
-<gazebo reference="camera_link">
-    <material></material>
-    <sensor name="camer_sensor" type="camera">
-        <pose>0 0 0 0 0 0</pose>
-        <visualize>true</visualize>
-        <update_rate>10.0</update_rate>
-        <plugin name="camera_controller" filename="libgazebo_ros_camera.so">
-           <frame_name>camera_link</frame_name>
-        </plugin>
-    </sensor>
-</gazebo>
+        <material>Gazebo/Red</material>
+        <sensor name="laser" type="ray">
+            <pose> 0 0 0 0 0 0 </pose>
+            <visualize>true</visualize>
+            <update_rate>10</update_rate>
+            <ray>
+                <scan>
+                    <horizontal>
+                        <samples>360</samples>
+                        <min_angle>-3.14</min_angle>
+                        <max_angle>3.14</max_angle>
+                    </horizontal>
+                </scan>
+                <range>
+                    <min>0.3</min>
+                    <max>12</max>
+                </range>
+            </ray>
+            <plugin name="laser_controller" filename="libgazebo_ros_ray_sensor.so">
+                <ros>
+                    <argument>~/out:=scan</argument>
+                </ros>
+                <output_type>sensor_msgs/LaserScan</output_type>
+                <frame_name>Laser_link</frame_name>
+            </plugin>
+        </sensor>
+    </gazebo>
+    <gazebo reference="camera_link">
+      <material></material>
+      <sensor name="camer_sensor" type="camera">
+          <pose>0 0 0 0 0 0</pose>
+          <visualize>true</visualize>
+          <update_rate>10.0</update_rate>
+          <plugin name="camera_controller" filename="libgazebo_ros_camera.so">
+             <frame_name>camera_link</frame_name>
+          </plugin>
+      </sensor>
+  </gazebo>
 </robot>
